Commit message: Update urdf to reflect the xacro file

File: stomp_test_support/urdf/test_kr210l150.urdf (robot description, URDF)
Before this commit: robot test_kr210, 12 links, 11 joints
Links:
- added link obstacle_cube; collision mesh filename=package://stomp_test_support/meshes/cube/visual/menger_spon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; visual mesh filename=package://stomp_test_support/meshes/cube/visual/menger_spon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
Joints:
- added joint world_to_cube: type fixed, parent world, child obstacle_cube, origin xyz=0.25 1.25 0.25
