Commit message: modified the collision geometry so that it encompases the space between the fingers

File: stomp_test_support/urdf/simple_2fgripper_macro.xacro (robot description, xacro)
@@ -25,10 +25,4 @@
 			</geometry>
 		</visual>
-		<collision>
-			<origin xyz="${0.5*workrange + 0.5*finger_thickness} 0 ${gripper_height + 0.5*finger_length}" rpy="0 0 0"/>
-			<geometry>
-				<box size="${finger_thickness} ${finger_width} ${finger_length}"/>
-			</geometry>
-		</collision>
 		<visual>
 			<material name="black"/>
@@ -39,7 +33,7 @@
 		</visual>
 		<collision>
-			<origin xyz="-${0.5*workrange + 0.5*finger_thickness} 0 ${gripper_height + 0.5*finger_length}" rpy="0 0 0"/>
+			<origin xyz="0 0 ${gripper_height + 0.5*finger_length}" rpy="0 0 0"/>
 			<geometry>
-				<box size="${finger_thickness} ${finger_width} ${finger_length}"/>
+				<box size="${finger_thickness + workrange} ${finger_width} ${finger_length}"/>
 			</geometry>
 		</collision>
