Commit message: added rail with a prismatic joint to the robot base in the test_kr210l150 workcell

File: stomp_test_support/urdf/test_kr210l150.xacro (robot description, xacro)
@@ -4,5 +4,26 @@
 	<xacro:include filename="$(find stomp_test_support)/urdf/kr210l150_macro.xacro"/>
 	<xacro:kuka_kr210l150 prefix=""/>
+  <xacro:property name="rail_cross_section" value="0.1"/>
   <link name="world"/>
+  <link name="rail">
+    <visual>
+      <origin xyz="0 0 0"/>
+      <geometry>
+        <box size="4 ${rail_cross_section} ${rail_cross_section}"/>
+      </geometry>
+      <material name="yellow">
+       <color rgba="1.0 1.0 0 1.0"/>
+      </material>
+    </visual>
+    <collision>
+      <origin xyz="0 0 0"/>
+      <geometry>
+        <box size="4 0.1 0.1"/>
+      </geometry>
+      <material name="yellow">
+       <color rgba="1.0 1.0 0 1.0"/>
+      </material>
+    </collision>
+  </link>
   <xacro:property name="cylinder_height" value="8.0"/>
   <link name="obstacle_cylinder">
@@ -26,8 +47,15 @@
     </collision>
   </link>
-  <joint name="world_to_base" type="fixed">
+  <joint name="world_to_rails" type="fixed">
     <parent link="world" />
+    <child link="rail" />
+    <origin xyz="0 0 0"/>
+  </joint>
+  <joint name="rail_to_base" type="prismatic">
+    <parent link="rail" />
     <child link="base_link" />
-    <origin xyz="0 0 0"/>
+    <origin xyz="0 0 ${0.5*rail_cross_section}"/>
+    <axis xyz="1 0 0"/>
+    <limit lower="-2" upper="2" effort="1" velocity="1"/>
   </joint>
   <joint name="world_to_cylinder" type="fixed">

Commit message: added walls to the workcell of the test robot for stomp

File: stomp_test_support/urdf/test_kr210l150.xacro (robot description, xacro)
@@ -5,5 +5,101 @@
 	<xacro:kuka_kr210l150 prefix=""/>
   <xacro:property name="rail_cross_section" value="0.1"/>
+  <xacro:property name="workcell_width" value="5.0"/>
+  <xacro:property name="workcell_length" value="8.0"/>
+  <xacro:property name="workcell_height" value="3.0"/>
+  <xacro:property name="workcell_thickness" value="0.01"/>
+  <xacro:property name="workcell_z" value="-0.1"/>
   <link name="world"/>
+  <material name="workcell_material">
+   <color rgba="0.8 1.0 0.8 0.2"/>
+  </material>
+  <link name="workcell_bounds">
+    <!-- visual geometries -->
+    <!--<visual> --><!-- top -->
+    <!-- <origin xyz="0 0 ${workcell_height}"/>
+      <geometry>
+        <box size="${workcell_length} ${workcell_width} ${workcell_thickness}"/>
+      </geometry>
+      <material name="workcell_material"/>
+    </visual> -->
+    <visual><!-- right ( +x ) -->
+      <origin xyz="${0.5*workcell_length} 0 ${0.5*workcell_height}"/>
+      <geometry>
+        <box size="${workcell_thickness} ${workcell_width} ${workcell_height}"/>
+      </geometry>
+      <material name="workcell_material"/>
+    </visual>
+    <visual><!-- bottom -->
+      <material name="workcell_material"/>
+      <origin xyz="0 0 0"/>
+      <geometry>
+        <box size="${workcell_length} ${workcell_width} ${workcell_thickness}"/>
+      </geometry>
+    </visual>
+    <visual><!-- left ( -x ) -->
+      <origin xyz="${-0.5*workcell_length} 0 ${0.5*workcell_height}"/>
+      <geometry>
+        <box size="${workcell_thickness} ${workcell_width} ${workcell_height}"/>
+      </geometry>
+      <material name="workcell_material"/>
+    </visual>
+    <!--<visual>--> <!-- front ( +y ) -->
+      <!--<origin xyz="0 ${0.5*workcell_width} ${0.5*workcell_height}"/>
+      <geometry>
+        <box size="${workcell_length} ${workcell_thickness} ${workcell_height}"/>
+      </geometry>
+      <material name="workcell_material"/>
+    </visual>-->
+    <visual><!-- rear ( -y ) -->
+      <origin xyz="0 ${-0.5*workcell_width} ${0.5*workcell_height}"/>
+      <geometry>
+        <box size="${workcell_length} ${workcell_thickness} ${workcell_height}"/>
+      </geometry>
+      <material name="workcell_material"/>
+    </visual>
+    <!-- collision geometries -->
+    <collision><!-- top -->
+      <origin xyz="0 0 ${workcell_height}"/>
+      <geometry>
+        <box size="${workcell_length} ${workcell_width} ${workcell_thickness}"/>
+      </geometry>
+      <material name="workcell_material"/>
+    </collision>
+    <collision><!-- right ( +x ) -->
+      <origin xyz="${0.5*workcell_length} 0 ${0.5*workcell_height}"/>
+      <geometry>
+        <box size="${workcell_thickness} ${workcell_width} ${workcell_height}"/>
+      </geometry>
+      <material name="workcell_material"/>
+    </collision>
+    <collision><!-- bottom -->
+      <material name="workcell_material"/>
+      <origin xyz="0 0 0"/>
+      <geometry>
+        <box size="${workcell_length} ${workcell_width} ${workcell_thickness}"/>
+      </geometry>
+    </collision>
+    <collision><!-- left ( -x ) -->
+      <origin xyz="${-0.5*workcell_length} 0 ${0.5*workcell_height}"/>
+      <geometry>
+        <box size="${workcell_thickness} ${workcell_width} ${workcell_height}"/>
+      </geometry>
+      <material name="workcell_material"/>
+    </collision>
+    <collision><!-- front ( +y ) -->
+      <origin xyz="0 ${0.5*workcell_width} ${0.5*workcell_height}"/>
+      <geometry>
+        <box size="${workcell_length} ${workcell_thickness} ${workcell_height}"/>
+      </geometry>
+      <material name="workcell_material"/>
+    </collision>
+    <collision><!-- rear ( -y ) -->
+      <origin xyz="0 ${-0.5*workcell_width} ${0.5*workcell_height}"/>
+      <geometry>
+        <box size="${workcell_length} ${workcell_thickness} ${workcell_height}"/>
+      </geometry>
+      <material name="workcell_material"/>
+    </collision>
+  </link>
   <link name="rail">
     <visual>
@@ -47,4 +143,9 @@
     </collision>
   </link>
+  <joint name="world_to_bounds" type="fixed">
+    <parent link="world" />
+    <child link="workcell_bounds" />
+    <origin xyz="0 0 ${workcell_z}"/>
+  </joint>
   <joint name="world_to_rails" type="fixed">
     <parent link="world" />

Commit message: Add mesh with 500K triangles

File: stomp_test_support/urdf/test_kr210l150.xacro (robot description, xacro)
@@ -143,4 +143,24 @@
     </collision>
   </link>
+  <link name="obstacle_cube">
+    <visual>
+      <origin xyz="0 0 0"/>
+      <geometry>
+        <mesh filename="package://stomp_test_support/meshes/cube/visual/menger_sponge.stl"/>
+      </geometry>
+     <material name="red">
+       <color rgba="1.0 0.4 0.4 1.0"/>
+     </material>
+    </visual>
+    <collision>
+      <origin xyz="0 0 0"/>
+      <geometry>
+        <mesh filename="package://stomp_test_support/meshes/cube/visual/menger_sponge.stl"/>
+      </geometry>
+     <material name="red">
+       <color rgba="1.0 0.4 0.4 1.0"/>
+     </material>
+    </collision>
+  </link>
   <joint name="world_to_bounds" type="fixed">
     <parent link="world" />
@@ -165,3 +185,8 @@
     <origin xyz="0 1.5 ${0.5*cylinder_height}"/>
   </joint>
+  <joint name="world_to_cube" type="fixed">
+    <parent link="world" />
+    <child link="obstacle_cube" />
+    <origin xyz="0.25 1.25 0.25"/>
+  </joint>
 </robot>

Commit message: Modify the test xacro to allow switching to a high triangle count version for profile testing

File: stomp_test_support/urdf/test_kr210l150.xacro (robot description, xacro)
@@ -1,192 +1,7 @@
 <?xml version="1.0" ?>
-<!--Generates a urdf from the macro in kr210_macro.xacro -->
 <robot name="test_kr210" xmlns:xacro="http://ros.org/wiki/xacro">
-	<xacro:include filename="$(find stomp_test_support)/urdf/kr210l150_macro.xacro"/>
-	<xacro:kuka_kr210l150 prefix=""/>
-  <xacro:property name="rail_cross_section" value="0.1"/>
-  <xacro:property name="workcell_width" value="5.0"/>
-  <xacro:property name="workcell_length" value="8.0"/>
-  <xacro:property name="workcell_height" value="3.0"/>
-  <xacro:property name="workcell_thickness" value="0.01"/>
-  <xacro:property name="workcell_z" value="-0.1"/>
-  <link name="world"/>
-  <material name="workcell_material">
-   <color rgba="0.8 1.0 0.8 0.2"/>
-  </material>
-  <link name="workcell_bounds">
-    <!-- visual geometries -->
-    <!--<visual> --><!-- top -->
-    <!-- <origin xyz="0 0 ${workcell_height}"/>
-      <geometry>
-        <box size="${workcell_length} ${workcell_width} ${workcell_thickness}"/>
-      </geometry>
-      <material name="workcell_material"/>
-    </visual> -->
-    <visual><!-- right ( +x ) -->
-      <origin xyz="${0.5*workcell_length} 0 ${0.5*workcell_height}"/>
-      <geometry>
-        <box size="${workcell_thickness} ${workcell_width} ${workcell_height}"/>
-      </geometry>
-      <material name="workcell_material"/>
-    </visual>
-    <visual><!-- bottom -->
-      <material name="workcell_material"/>
-      <origin xyz="0 0 0"/>
-      <geometry>
-        <box size="${workcell_length} ${workcell_width} ${workcell_thickness}"/>
-      </geometry>
-    </visual>
-    <visual><!-- left ( -x ) -->
-      <origin xyz="${-0.5*workcell_length} 0 ${0.5*workcell_height}"/>
-      <geometry>
-        <box size="${workcell_thickness} ${workcell_width} ${workcell_height}"/>
-      </geometry>
-      <material name="workcell_material"/>
-    </visual>
-    <!--<visual>--> <!-- front ( +y ) -->
-      <!--<origin xyz="0 ${0.5*workcell_width} ${0.5*workcell_height}"/>
-      <geometry>
-        <box size="${workcell_length} ${workcell_thickness} ${workcell_height}"/>
-      </geometry>
-      <material name="workcell_material"/>
-    </visual>-->
-    <visual><!-- rear ( -y ) -->
-      <origin xyz="0 ${-0.5*workcell_width} ${0.5*workcell_height}"/>
-      <geometry>
-        <box size="${workcell_length} ${workcell_thickness} ${workcell_height}"/>
-      </geometry>
-      <material name="workcell_material"/>
-    </visual>
-    <!-- collision geometries -->
-    <collision><!-- top -->
-      <origin xyz="0 0 ${workcell_height}"/>
-      <geometry>
-        <box size="${workcell_length} ${workcell_width} ${workcell_thickness}"/>
-      </geometry>
-      <material name="workcell_material"/>
-    </collision>
-    <collision><!-- right ( +x ) -->
-      <origin xyz="${0.5*workcell_length} 0 ${0.5*workcell_height}"/>
-      <geometry>
-        <box size="${workcell_thickness} ${workcell_width} ${workcell_height}"/>
-      </geometry>
-      <material name="workcell_material"/>
-    </collision>
-    <collision><!-- bottom -->
-      <material name="workcell_material"/>
-      <origin xyz="0 0 0"/>
-      <geometry>
-        <box size="${workcell_length} ${workcell_width} ${workcell_thickness}"/>
-      </geometry>
-    </collision>
-    <collision><!-- left ( -x ) -->
-      <origin xyz="${-0.5*workcell_length} 0 ${0.5*workcell_height}"/>
-      <geometry>
-        <box size="${workcell_thickness} ${workcell_width} ${workcell_height}"/>
-      </geometry>
-      <material name="workcell_material"/>
-    </collision>
-    <collision><!-- front ( +y ) -->
-      <origin xyz="0 ${0.5*workcell_width} ${0.5*workcell_height}"/>
-      <geometry>
-        <box size="${workcell_length} ${workcell_thickness} ${workcell_height}"/>
-      </geometry>
-      <material name="workcell_material"/>
-    </collision>
-    <collision><!-- rear ( -y ) -->
-      <origin xyz="0 ${-0.5*workcell_width} ${0.5*workcell_height}"/>
-      <geometry>
-        <box size="${workcell_length} ${workcell_thickness} ${workcell_height}"/>
-      </geometry>
-      <material name="workcell_material"/>
-    </collision>
-  </link>
-  <link name="rail">
-    <visual>
-      <origin xyz="0 0 0"/>
-      <geometry>
-        <box size="4 ${rail_cross_section} ${rail_cross_section}"/>
-      </geometry>
-      <material name="yellow">
-       <color rgba="1.0 1.0 0 1.0"/>
-      </material>
-    </visual>
-    <collision>
-      <origin xyz="0 0 0"/>
-      <geometry>
-        <box size="4 0.1 0.1"/>
-      </geometry>
-      <material name="yellow">
-       <color rgba="1.0 1.0 0 1.0"/>
-      </material>
-    </collision>
-  </link>
-  <xacro:property name="cylinder_height" value="8.0"/>
-  <link name="obstacle_cylinder">
-    <visual>
-      <origin xyz="0 0 0"/>
-      <geometry>
-        <cylinder radius="0.2" length="${cylinder_height}"/>
-      </geometry>
-     <material name="cyan">
-       <color rgba="0 1.0 1.0 1.0"/>
-     </material>
-    </visual>
-    <collision>
-      <origin xyz="0 0 0"/>
-      <geometry>
-        <cylinder radius="0.2" length="${cylinder_height}"/>
-      </geometry>
-     <material name="cyan">
-       <color rgba="0 1.0 1.0 1.0"/>
-     </material>
-    </collision>
-  </link>
-  <link name="obstacle_cube">
-    <visual>
-      <origin xyz="0 0 0"/>
-      <geometry>
-        <mesh filename="package://stomp_test_support/meshes/cube/visual/menger_sponge.stl"/>
-      </geometry>
-     <material name="red">
-       <color rgba="1.0 0.4 0.4 1.0"/>
-     </material>
-    </visual>
-    <collision>
-      <origin xyz="0 0 0"/>
-      <geometry>
-        <mesh filename="package://stomp_test_support/meshes/cube/visual/menger_sponge.stl"/>
-      </geometry>
-     <material name="red">
-       <color rgba="1.0 0.4 0.4 1.0"/>
-     </material>
-    </collision>
-  </link>
-  <joint name="world_to_bounds" type="fixed">
-    <parent link="world" />
-    <child link="workcell_bounds" />
-    <origin xyz="0 0 ${workcell_z}"/>
-  </joint>
-  <joint name="world_to_rails" type="fixed">
-    <parent link="world" />
-    <child link="rail" />
-    <origin xyz="0 0 0"/>
-  </joint>
-  <joint name="rail_to_base" type="prismatic">
-    <parent link="rail" />
-    <child link="base_link" />
-    <origin xyz="0 0 ${0.5*rail_cross_section}"/>
-    <axis xyz="1 0 0"/>
-    <limit lower="-2" upper="2" effort="1" velocity="1"/>
-  </joint>
-  <joint name="world_to_cylinder" type="fixed">
-    <parent link="world" />
-    <child link="obstacle_cylinder" />
-    <origin xyz="0 1.5 ${0.5*cylinder_height}"/>
-  </joint>
-  <joint name="world_to_cube" type="fixed">
-    <parent link="world" />
-    <child link="obstacle_cube" />
-    <origin xyz="0.25 1.25 0.25"/>
-  </joint>
+  <xacro:include filename="$(find stomp_test_support)/urdf/kr210l150_macro.xacro"/>
+  <xacro:kuka_kr210l150 prefix=""/>
+  <xacro:include filename="$(find stomp_test_support)/urdf/test_kr210l150_macro.xacro"/>
+  <xacro:test_kr210l150 simple="true"/>
 </robot>

File: stomp_test_support/urdf/test_kr210l150_simple.urdf (robot description, URDF)
Before this commit: robot test_kr210, 13 links, 12 joints
Links:
- removed link obstacle_cube
Joints:
- removed joint world_to_cube

Commit message: added simple 2 finger gripper

File: stomp_test_support/urdf/test_kr210l150.xacro (robot description, xacro)
@@ -5,3 +5,10 @@
   <xacro:include filename="$(find stomp_test_support)/urdf/test_kr210l150_macro.xacro"/>
   <xacro:test_kr210l150 simple="true"/>
+  <xacro:include filename="$(find stomp_test_support)/urdf/simple_2fgripper_macro.xacro"/>
+  <xacro:simple_2fgripper_link prefix=""/>
+  <joint name="wrist_to_gripper" type="fixed">
+    <parent link="tool0" />
+    <child link="gripper_frame" />
+    <origin xyz="0 0 0" rpy="0 1.57079632679 0"/>
+  </joint>
 </robot>
