Commit message: xacro tags should be prepended with 'xacro' xml namespace

File: stomp_test_support/urdf/kr210l150_macro.xacro (robot description, xacro)
@@ -1,5 +1,5 @@
 <robot xmlns:xacro="http://wiki.ros.org/xacro">
-	<property name="pi" value="3.141592654" />
-	<property name="deg" value="0.017453293" /> <!--degrees to radians-->
+	<xacro:property name="pi" value="3.141592654" />
+	<xacro:property name="deg" value="0.017453293" /> <!--degrees to radians-->
 	<xacro:macro name="kuka_kr210l150" params="prefix">
   <link

Commit message: remove redefined pi

File: stomp_test_support/urdf/kr210l150_macro.xacro (robot description, xacro)
@@ -1,4 +1,3 @@
 <robot xmlns:xacro="http://wiki.ros.org/xacro">
-	<xacro:property name="pi" value="3.141592654" />
 	<xacro:property name="deg" value="0.017453293" /> <!--degrees to radians-->
 	<xacro:macro name="kuka_kr210l150" params="prefix">

Commit message: Update of xacro command and format (#72)
* update xmlnx:xacro

* xacro tags should be prepended with 'xacro' xml namespace

* use xacro instead

* add --inorder option

* remove redefined pi

File: stomp_test_support/urdf/kr210l150_macro.xacro (robot description, xacro)
@@ -1,5 +1,4 @@
-<robot xmlns:xacro="http://ros.org/wiki/xacro">
-	<property name="pi" value="3.141592654" />
-	<property name="deg" value="0.017453293" /> <!--degrees to radians-->
+<robot xmlns:xacro="http://wiki.ros.org/xacro">
+	<xacro:property name="deg" value="0.017453293" /> <!--degrees to radians-->
 	<xacro:macro name="kuka_kr210l150" params="prefix">
   <link
