Commit message: moved industrial_moveit_benchmarking resource files into that package

File: industrial_moveit_benchmarking/resources/urdf/test_kr210l150_500K.urdf (robot description, URDF)
Before this commit: robot test_kr210, 12 links, 11 joints
Links:
- added link obstacle_cube; collision mesh filename=package://industrial_moveit_benchmarking/resources/meshes/v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; visual mesh filename=package://industrial_moveit_benchmarking/resources/meshes/v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
Joints:
- added joint world_to_cube: type fixed, parent world, child obstacle_cube, origin xyz=0.25 1.25 0.25

Commit message: renamed stomp_test_support to industrial_moveit_test_support

File: industrial_moveit_benchmarking/resources/urdf/test_kr210l150_500K.urdf (robot description, URDF)
Before this commit: robot test_kr210, 13 links, 12 joints
Links:
- link Link1: geometry collision mesh filename=package://industrial_moveit_test_support/meshes/kr210l150/c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; visual mesh filename=package://industrial_moveit_test_support/meshes/kr210l150/v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
- link base_link: geometry collision mesh filename=package://industrial_moveit_test_support/meshes/kr210l150/c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; visual mesh filename=package://industrial_moveit_test_support/meshes/kr210l150/v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
- link link_2: geometry collision mesh filename=package://industrial_moveit_test_support/meshes/kr210l150/c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; visual mesh filename=package://industrial_moveit_test_support/meshes/kr210l150/v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
- link link_3: geometry collision mesh filename=package://industrial_moveit_test_support/meshes/kr210l150/c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; visual mesh filename=package://industrial_moveit_test_support/meshes/kr210l150/v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
- link link_4: geometry collision mesh filename=package://industrial_moveit_test_support/meshes/kr210l150/c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; visual mesh filename=package://industrial_moveit_test_support/meshes/kr210l150/v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
- link link_5: geometry collision mesh filename=package://industrial_moveit_test_support/meshes/kr210l150/c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; visual mesh filename=package://industrial_moveit_test_support/meshes/kr210l150/v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
- link link_6: geometry collision mesh filename=package://industrial_moveit_test_support/meshes/kr210l150/c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; visual mesh filename=package://industrial_moveit_test_support/meshes/kr210l150/v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

File: industrial_moveit_test_support/urdf/kr210l150_macro.xacro (robot description, xacro)
@@ -24,19 +24,19 @@
       <geometry>
         <mesh
-          filename="package://stomp_test_support/meshes/kr210l150/visual/base_link.dae" />
-      </geometry>
-      <material
-        name="">
-        <color
-          rgba="0.75294 0.75294 0.75294 1" />
-      </material>
-    </visual>
-    <collision>
-      <origin
-        xyz="0 0 0"
-        rpy="${-pi/2} 0 0" />
-      <geometry>
-        <mesh
-          filename="package://stomp_test_support/meshes/kr210l150/collision/base_link.stl" />
+          filename="package://industrial_moveit_test_support/meshes/kr210l150/visual/base_link.dae" />
+      </geometry>
+      <material
+        name="">
+        <color
+          rgba="0.75294 0.75294 0.75294 1" />
+      </material>
+    </visual>
+    <collision>
+      <origin
+        xyz="0 0 0"
+        rpy="${-pi/2} 0 0" />
+      <geometry>
+        <mesh
+          filename="package://industrial_moveit_test_support/meshes/kr210l150/collision/base_link.stl" />
       </geometry>
     </collision>
@@ -64,19 +64,19 @@
       <geometry>
         <mesh
-          filename="package://stomp_test_support/meshes/kr210l150/visual/link_1.dae" />
-      </geometry>
-      <material
-        name="">
-        <color
-          rgba="0.75294 0.75294 0.75294 1" />
-      </material>
-    </visual>
-    <collision>
-      <origin
-        xyz="0 0 0"
-        rpy="0 0 0" />
-      <geometry>
-        <mesh
-          filename="package://stomp_test_support/meshes/kr210l150/collision/link_1.stl" />
+          filename="package://industrial_moveit_test_support/meshes/kr210l150/visual/link_1.dae" />
+      </geometry>
+      <material
+        name="">
+        <color
+          rgba="0.75294 0.75294 0.75294 1" />
+      </material>
+    </visual>
+    <collision>
+      <origin
+        xyz="0 0 0"
+        rpy="0 0 0" />
+      <geometry>
+        <mesh
+          filename="package://industrial_moveit_test_support/meshes/kr210l150/collision/link_1.stl" />
       </geometry>
     </collision>
@@ -118,19 +118,19 @@
       <geometry>
         <mesh
-          filename="package://stomp_test_support/meshes/kr210l150/visual/link_2.dae" />
-      </geometry>
-      <material
-        name="">
-        <color
-          rgba="0.75294 0.75294 0.75294 1" />
-      </material>
-    </visual>
-    <collision>
-      <origin
-        xyz="0 0 0"
-        rpy="0 0 0" />
-      <geometry>
-        <mesh
-          filename="package://stomp_test_support/meshes/kr210l150/collision/link_2.stl" />
+          filename="package://industrial_moveit_test_support/meshes/kr210l150/visual/link_2.dae" />
+      </geometry>
+      <material
+        name="">
+        <color
+          rgba="0.75294 0.75294 0.75294 1" />
+      </material>
+    </visual>
+    <collision>
+      <origin
+        xyz="0 0 0"
+        rpy="0 0 0" />
+      <geometry>
+        <mesh
+          filename="package://industrial_moveit_test_support/meshes/kr210l150/collision/link_2.stl" />
       </geometry>
     </collision>
@@ -172,19 +172,19 @@
       <geometry>
         <mesh
-          filename="package://stomp_test_support/meshes/kr210l150/visual/link_3.dae" />
-      </geometry>
-      <material
-        name="">
-        <color
-          rgba="0.75294 0.75294 0.75294 1" />
-      </material>
-    </visual>
-    <collision>
-      <origin
-        xyz="0 0 0"
-        rpy="0 0 0" />
-      <geometry>
-        <mesh
-          filename="package://stomp_test_support/meshes/kr210l150/collision/link_3.stl" />
+          filename="package://industrial_moveit_test_support/meshes/kr210l150/visual/link_3.dae" />
+      </geometry>
+      <material
+        name="">
+        <color
+          rgba="0.75294 0.75294 0.75294 1" />
+      </material>
+    </visual>
+    <collision>
+      <origin
+        xyz="0 0 0"
+        rpy="0 0 0" />
+      <geometry>
+        <mesh
+          filename="package://industrial_moveit_test_support/meshes/kr210l150/collision/link_3.stl" />
       </geometry>
     </collision>
@@ -226,19 +226,19 @@
       <geometry>
         <mesh
-          filename="package://stomp_test_support/meshes/kr210l150/visual/link_4.dae" />
-      </geometry>
-      <material
-        name="">
-        <color
-          rgba="0.75294 0.75294 0.75294 1" />
-      </material>
-    </visual>
-    <collision>
-      <origin
-        xyz="0 0 0"
-        rpy="0 0 0" />
-      <geometry>
-        <mesh
-          filename="package://stomp_test_support/meshes/kr210l150/collision/link_4.stl" />
+          filename="package://industrial_moveit_test_support/meshes/kr210l150/visual/link_4.dae" />
+      </geometry>
+      <material
+        name="">
+        <color
+          rgba="0.75294 0.75294 0.75294 1" />
+      </material>
+    </visual>
+    <collision>
+      <origin
+        xyz="0 0 0"
+        rpy="0 0 0" />
+      <geometry>
+        <mesh
+          filename="package://industrial_moveit_test_support/meshes/kr210l150/collision/link_4.stl" />
       </geometry>
     </collision>
@@ -280,19 +280,19 @@
       <geometry>
         <mesh
-          filename="package://stomp_test_support/meshes/kr210l150/visual/link_5.dae" />
-      </geometry>
-      <material
-        name="">
-        <color
-          rgba="0.75294 0.75294 0.75294 1" />
-      </material>
-    </visual>
-    <collision>
-      <origin
-        xyz="0 0 0"
-        rpy="0 0 0" />
-      <geometry>
-        <mesh
-          filename="package://stomp_test_support/meshes/kr210l150/collision/link_5.stl" />
+          filename="package://industrial_moveit_test_support/meshes/kr210l150/visual/link_5.dae" />
+      </geometry>
+      <material
+        name="">
+        <color
+          rgba="0.75294 0.75294 0.75294 1" />
+      </material>
+    </visual>
+    <collision>
+      <origin
+        xyz="0 0 0"
+        rpy="0 0 0" />
+      <geometry>
+        <mesh
+          filename="package://industrial_moveit_test_support/meshes/kr210l150/collision/link_5.stl" />
       </geometry>
     </collision>
@@ -334,19 +334,19 @@
       <geometry>
         <mesh
-          filename="package://stomp_test_support/meshes/kr210l150/visual/link_6.dae" />
-      </geometry>
-      <material
-        name="">
-        <color
-          rgba="0.75294 0.75294 0.75294 1" />
-      </material>
-    </visual>
-    <collision>
-      <origin
-        xyz="0 0 0"
-        rpy="0 0 0" />
-      <geometry>
-        <mesh
-          filename="package://stomp_test_support/meshes/kr210l150/collision/link_6.stl" />
+          filename="package://industrial_moveit_test_support/meshes/kr210l150/visual/link_6.dae" />
+      </geometry>
+      <material
+        name="">
+        <color
+          rgba="0.75294 0.75294 0.75294 1" />
+      </material>
+    </visual>
+    <collision>
+      <origin
+        xyz="0 0 0"
+        rpy="0 0 0" />
+      <geometry>
+        <mesh
+          filename="package://industrial_moveit_test_support/meshes/kr210l150/collision/link_6.stl" />
       </geometry>
     </collision>

File: industrial_moveit_test_support/urdf/test_kr210l150.xacro (robot description, xacro)
@@ -1,9 +1,9 @@
 <?xml version="1.0" ?>
 <robot name="test_kr210" xmlns:xacro="http://wiki.ros.org/xacro">
-  <xacro:include filename="$(find stomp_test_support)/urdf/kr210l150_macro.xacro"/>
+  <xacro:include filename="$(find industrial_moveit_test_support)/urdf/kr210l150_macro.xacro"/>
   <xacro:kuka_kr210l150 prefix=""/>
-  <xacro:include filename="$(find stomp_test_support)/urdf/test_kr210l150_macro.xacro"/>
+  <xacro:include filename="$(find industrial_moveit_test_support)/urdf/test_kr210l150_macro.xacro"/>
   <xacro:test_kr210l150 simple="true"/>
-  <xacro:include filename="$(find stomp_test_support)/urdf/simple_2fgripper_macro.xacro"/>
+  <xacro:include filename="$(find industrial_moveit_test_support)/urdf/simple_2fgripper_macro.xacro"/>
   <xacro:simple_2fgripper_link prefix=""/>
   <joint name="wrist_to_gripper" type="fixed">

File: industrial_moveit_test_support/urdf/test_kr210l150_macro.xacro (robot description, xacro)
@@ -147,5 +147,5 @@
         <origin xyz="0 0 0"/>
         <geometry>
-          <mesh filename="package://stomp_test_support/meshes/cube/visual/menger_sponge.stl"/>
+          <mesh filename="package://industrial_moveit_test_support/meshes/cube/visual/menger_sponge.stl"/>
         </geometry>
        <material name="red">
@@ -156,5 +156,5 @@
         <origin xyz="0 0 0"/>
         <geometry>
-          <mesh filename="package://stomp_test_support/meshes/cube/visual/menger_sponge.stl"/>
+          <mesh filename="package://industrial_moveit_test_support/meshes/cube/visual/menger_sponge.stl"/>
         </geometry>
        <material name="red">
